Commit message: add imu_link

File: custom_pkgs/locobot/urdf/imu.urdf.xacro (robot description, xacro)
@@ -11,12 +11,11 @@
         <origin xyz="0 0 0" rpy="0 0 0"/>
         <geometry>
-          <box size="0.05 0.05 0.05"/> <!-- Placeholder dimensions, adjust as needed -->
+          <box size="0.01 0.01 0.01"/> <!-- Placeholder dimensions, adjust as needed -->
         </geometry>
-        <material name="grey"/>
       </visual>
     </link>
     <!-- Fixed Joint to Attach IMU to the Robot -->
     <joint name="${robot_name}/${imu_link_name}_joint" type="fixed">
-      <origin xyz="0.1 0 0.05" rpy="0 0 ${pi}"/> <!-- Adjust xyz and rpy based on the desired position and orientation -->
+      <origin xyz="-0.04 -0.09 -0.01" rpy="0 0 0"/> <!-- Adjust xyz and rpy based on the desired position and orientation -->
       <parent link="${robot_name}/${imu_parent_link}"/>
       <child link="${robot_name}/${imu_link_name}"/>

Commit message: update

File: custom_pkgs/locobot/urdf/imu.urdf.xacro (robot description, xacro)
@@ -17,5 +17,5 @@
     <!-- Fixed Joint to Attach IMU to the Robot -->
     <joint name="${robot_name}/${imu_link_name}_joint" type="fixed">
-      <origin xyz="-0.04 -0.09 -0.01" rpy="0 0 0"/> <!-- Adjust xyz and rpy based on the desired position and orientation -->
+      <origin xyz="-0.14477 -0.031 0.24" rpy="0 0 0"/> <!-- Adjust xyz and rpy based on the desired position and orientation -->
       <parent link="${robot_name}/${imu_parent_link}"/>
       <child link="${robot_name}/${imu_link_name}"/>

File: interbotix_ros_rovers/interbotix_ros_xslocobots/interbotix_xslocobot_descriptions/urdf/locobot.urdf.xacro (robot description, xacro)
@@ -26,5 +26,5 @@
   <xacro:include filename="$(find interbotix_xslocobot_descriptions)/urdf/pan_and_tilt.urdf.xacro" />
   <xacro:include filename="$(find locobot)/urdf/imu.urdf.xacro"/>
-  <xacro:imu robot_name="locobot" imu_link_name="imu_link" imu_parent_link="laser_frame_link"/>
+  <xacro:imu robot_name="locobot" imu_link_name="imu_link" imu_parent_link="base_footprint"/>
   <link name="$(arg robot_name)/base_footprint"/>
   <xacro:if value="${arm_type == 'mobile_wx250s'}">

Commit message: update imu and lidar urdf

File: custom_pkgs/locobot/urdf/imu.urdf.xacro (robot description, xacro)
@@ -17,5 +17,5 @@
     <!-- Fixed Joint to Attach IMU to the Robot -->
     <joint name="${robot_name}/${imu_link_name}_joint" type="fixed">
-      <origin xyz="-0.14477 -0.031 0.24" rpy="0 0 0"/> <!-- Adjust xyz and rpy based on the desired position and orientation -->
+      <origin xyz="-0.14962 -0.078 0.25" rpy="0 0 0"/> <!-- Adjust xyz and rpy based on the desired position and orientation -->
       <parent link="${robot_name}/${imu_parent_link}"/>
       <child link="${robot_name}/${imu_link_name}"/>

File: interbotix_ros_rovers/interbotix_ros_xslocobots/interbotix_xslocobot_descriptions/urdf/lidar.urdf.xacro (robot description, xacro)
@@ -33,14 +33,14 @@
       <disableFixedJointLumping>true</disableFixedJointLumping>
     </gazebo>
-    <joint name="lidar" type="fixed">
+    <!-- <joint name="lidar" type="fixed">
       <origin rpy="0 0 ${pi}" xyz="0 0 0.09425"/>
       <parent link="$(arg robot_name)/lidar_tower_link"/>
       <child link="$(arg robot_name)/laser_frame_link"/>
-    </joint>
-    <!-- <joint name="lidar" type="fixed">
-      <origin rpy="0 0 0" xyz="-0.09544 0 0.24"/>
+    </joint> -->
+    <joint name="lidar" type="fixed">
+      <origin rpy="0 0 0" xyz="-0.09277 0 0.26"/>
       <parent link="$(arg robot_name)/base_footprint"/>
       <child link="$(arg robot_name)/laser_frame_link"/>
-    </joint> -->
+    </joint>
     <gazebo reference="lidar">
       <disableFixedJointLumping>true</disableFixedJointLumping>

Commit message: refactor launch files

File: custom_pkgs/locobot/urdf/imu.urdf.xacro (robot description, xacro)
@@ -17,5 +17,5 @@
     <!-- Fixed Joint to Attach IMU to the Robot -->
     <joint name="${robot_name}/${imu_link_name}_joint" type="fixed">
-      <origin xyz="-0.14962 -0.078 0.25" rpy="0 0 0"/> <!-- Adjust xyz and rpy based on the desired position and orientation -->
+      <origin xyz="-0.14962 -0.078 0.242" rpy="0 0 0"/> <!-- Adjust xyz and rpy based on the desired position and orientation -->
       <parent link="${robot_name}/${imu_parent_link}"/>
       <child link="${robot_name}/${imu_link_name}"/>

File: interbotix_ros_rovers/interbotix_ros_xslocobots/interbotix_xslocobot_descriptions/urdf/lidar.urdf.xacro (robot description, xacro)
@@ -39,5 +39,5 @@
     </joint> -->
     <joint name="lidar" type="fixed">
-      <origin rpy="0 0 0" xyz="-0.09277 0 0.26"/>
+      <origin rpy="0 0 0" xyz="-0.09277 0 0.25"/>
       <parent link="$(arg robot_name)/base_footprint"/>
       <child link="$(arg robot_name)/laser_frame_link"/>
